File: TicTacToeV1.kicad_pcb (KiCad board)
At the start: 2 copper layers, 64 x 87 mm, 34 parts, among them U1 74HC165, U2 74HC165, U3 MAX7219

Commit message: Updated for production by OSHPARK
Parts:
- S1, S10, S2, S3, S4, S5, S6, S7, S8, S9: footprint TicTacToeV1:B3W9000RG2C -> TicTacToeV1:B3W-9000-RG2C
