File: TicTacToeV1.kicad_sch (KiCad schematic)
At the start: 34 parts, among them U1 74HC165, U2 74HC165, U3 MAX7219

Commit message: Updated for production by OSHPARK
Parts:
- S1, S10, S2, S3, S4, S5, S6, S7, S8, S9: footprint TicTacToeV1:B3W9000RG2C -> TicTacToeV1:B3W-9000-RG2C
Changed lines of the file:
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@@
     (property "Reference" "S9" (id 0) (at 318.77 109.22 0))
     (property "Value" "B3W-9000-RG2C" (id 1) (at 318.77 111.76 0))
-    (property "Footprint" "TicTacToeV1:B3W9000RG2C" (id 2) (at 331.47 114.3 0)
+    (property "Footprint" "TicTacToeV1:B3W-9000-RG2C" (id 2) (at 331.47 114.3 0)
       (effects (font (size 1.27 1.27)) (justify left) hide)
     )
@@
     (property "Reference" "S2" (id 0) (at 260.35 38.1 0))
     (property "Value" "B3W-9000-RG2C" (id 1) (at 260.35 40.64 0))
-    (property "Footprint" "TicTacToeV1:B3W9000RG2C" (id 2) (at 273.05 43.18 0)
+    (property "Footprint" "TicTacToeV1:B3W-9000-RG2C" (id 2) (at 273.05 43.18 0)
       (effects (font (size 1.27 1.27)) (justify left) hide)
     )
@@
     (property "Reference" "S6" (id 0) (at 318.77 73.66 0))
     (property "Value" "B3W-9000-RG2C" (id 1) (at 318.77 76.2 0))
-    (property "Footprint" "TicTacToeV1:B3W9000RG2C" (id 2) (at 331.47 78.74 0)
+    (property "Footprint" "TicTacToeV1:B3W-9000-RG2C" (id 2) (at 331.47 78.74 0)
       (effects (font (size 1.27 1.27)) (justify left) hide)
     )
@@
     (property "Reference" "S4" (id 0) (at 201.93 73.66 0))
     (property "Value" "B3W-9000-RG2C" (id 1) (at 201.93 76.2 0))
-    (property "Footprint" "TicTacToeV1:B3W9000RG2C" (id 2) (at 214.63 78.74 0)
+    (property "Footprint" "TicTacToeV1:B3W-9000-RG2C" (id 2) (at 214.63 78.74 0)
       (effects (font (size 1.27 1.27)) (justify left) hide)
     )
@@
     (property "Reference" "S8" (id 0) (at 260.35 109.22 0))
     (property "Value" "B3W-9000-RG2C" (id 1) (at 260.35 111.76 0))
-    (property "Footprint" "TicTacToeV1:B3W9000RG2C" (id 2) (at 273.05 114.3 0)
+    (property "Footprint" "TicTacToeV1:B3W-9000-RG2C" (id 2) (at 273.05 114.3 0)
       (effects (font (size 1.27 1.27)) (justify left) hide)
     )
@@
     (property "Reference" "S5" (id 0) (at 260.35 73.66 0))
     (property "Value" "B3W-9000-RG2C" (id 1) (at 260.35 76.2 0))
-    (property "Footprint" "TicTacToeV1:B3W9000RG2C" (id 2) (at 273.05 78.74 0)
+    (property "Footprint" "TicTacToeV1:B3W-9000-RG2C" (id 2) (at 273.05 78.74 0)
       (effects (font (size 1.27 1.27)) (justify left) hide)
     )
@@
     (property "Reference" "S7" (id 0) (at 201.93 109.22 0))
     (property "Value" "B3W-9000-RG2C" (id 1) (at 201.93 111.76 0))
-    (property "Footprint" "TicTacToeV1:B3W9000RG2C" (id 2) (at 214.63 114.3 0)
+    (property "Footprint" "TicTacToeV1:B3W-9000-RG2C" (id 2) (at 214.63 114.3 0)
       (effects (font (size 1.27 1.27)) (justify left) hide)
     )
@@
     (property "Reference" "S10" (id 0) (at 63.5 26.67 0))
     (property "Value" "B3W-9000-RG2C" (id 1) (at 63.5 29.21 0))
-    (property "Footprint" "TicTacToeV1:B3W9000RG2C" (id 2) (at 76.2 31.75 0)
+    (property "Footprint" "TicTacToeV1:B3W-9000-RG2C" (id 2) (at 76.2 31.75 0)
       (effects (font (size 1.27 1.27)) (justify left) hide)
     )
@@
     (property "Reference" "S1" (id 0) (at 201.93 38.1 0))
     (property "Value" "B3W-9000-RG2C" (id 1) (at 201.93 40.64 0))
-    (property "Footprint" "TicTacToeV1:B3W9000RG2C" (id 2) (at 214.63 43.18 0)
+    (property "Footprint" "TicTacToeV1:B3W-9000-RG2C" (id 2) (at 214.63 43.18 0)
       (effects (font (size 1.27 1.27)) (justify left) hide)
     )
@@
     (property "Reference" "S3" (id 0) (at 318.77 38.1 0))
     (property "Value" "B3W-9000-RG2C" (id 1) (at 318.77 40.64 0))
-    (property "Footprint" "TicTacToeV1:B3W9000RG2C" (id 2) (at 331.47 43.18 0)
+    (property "Footprint" "TicTacToeV1:B3W-9000-RG2C" (id 2) (at 331.47 43.18 0)
       (effects (font (size 1.27 1.27)) (justify left) hide)
     )
@@
     )
     (path "/eb63f3b4-020d-4af5-94e0-4f1fb51c6526"
-      (reference "S1") (unit 1) (value "B3W-9000-RG2C") (footprint "TicTacToeV1:B3W9000RG2C")
+      (reference "S1") (unit 1) (value "B3W-9000-RG2C") (footprint "TicTacToeV1:B3W-9000-RG2C")
     )
     (path "/5d590629-c429-4026-ab75-9f4c561b4b05"
-      (reference "S2") (unit 1) (value "B3W-9000-RG2C") (footprint "TicTacToeV1:B3W9000RG2C")
+      (reference "S2") (unit 1) (value "B3W-9000-RG2C") (footprint "TicTacToeV1:B3W-9000-RG2C")
     )
     (path "/ecb602f8-02c5-4f83-ab9d-f6b307024336"
-      (reference "S3") (unit 1) (value "B3W-9000-RG2C") (footprint "TicTacToeV1:B3W9000RG2C")
+      (reference "S3") (unit 1) (value "B3W-9000-RG2C") (footprint "TicTacToeV1:B3W-9000-RG2C")
     )
     (path "/944e655b-ec2e-4d2c-9548-647572f3c62f"
-      (reference "S4") (unit 1) (value "B3W-9000-RG2C") (footprint "TicTacToeV1:B3W9000RG2C")
+      (reference "S4") (unit 1) (value "B3W-9000-RG2C") (footprint "TicTacToeV1:B3W-9000-RG2C")
     )
     (path "/a8eae4c4-7823-4a25-b017-e5ac7e09ba44"
-      (reference "S5") (unit 1) (value "B3W-9000-RG2C") (footprint "TicTacToeV1:B3W9000RG2C")
+      (reference "S5") (unit 1) (value "B3W-9000-RG2C") (footprint "TicTacToeV1:B3W-9000-RG2C")
     )
     (path "/78e4168a-1efa-4d36-8c45-69b733b5b2a2"
-      (reference "S6") (unit 1) (value "B3W-9000-RG2C") (footprint "TicTacToeV1:B3W9000RG2C")
+      (reference "S6") (unit 1) (value "B3W-9000-RG2C") (footprint "TicTacToeV1:B3W-9000-RG2C")
     )
     (path "/c9064f3e-7a3e-4139-bbeb-743e9ec9a3af"
-      (reference "S7") (unit 1) (value "B3W-9000-RG2C") (footprint "TicTacToeV1:B3W9000RG2C")
+      (reference "S7") (unit 1) (value "B3W-9000-RG2C") (footprint "TicTacToeV1:B3W-9000-RG2C")
     )
     (path "/95bd360d-cfc9-4ffe-b5fe-160e7e720aaa"
-      (reference "S8") (unit 1) (value "B3W-9000-RG2C") (footprint "TicTacToeV1:B3W9000RG2C")
+      (reference "S8") (unit 1) (value "B3W-9000-RG2C") (footprint "TicTacToeV1:B3W-9000-RG2C")
     )
     (path "/04927789-654c-4621-b2bd-76d08b095a5e"
-      (reference "S9") (unit 1) (value "B3W-9000-RG2C") (footprint "TicTacToeV1:B3W9000RG2C")
+      (reference "S9") (unit 1) (value "B3W-9000-RG2C") (footprint "TicTacToeV1:B3W-9000-RG2C")
     )
     (path "/d76e5a2d-126a-4af3-8aa3-754513d6e1a8"
-      (reference "S10") (unit 1) (value "B3W-9000-RG2C") (footprint "TicTacToeV1:B3W9000RG2C")
+      (reference "S10") (unit 1) (value "B3W-9000-RG2C") (footprint "TicTacToeV1:B3W-9000-RG2C")
     )
     (path "/dbc71d4d-2c11-4334-bd2a-0bb81daf8470"
