File: KiCAD/TicTacToeV1.kicad_sch (KiCad schematic)
At the start: 34 parts, among them U1 74HC165, U2 74HC165, U3 MAX7219

Commit message: Updated the register value based on the prototyping on the breadboard.
Parts:
- R11: value 330 -> 220
Changed lines of the file:
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@@
     (in_bom yes) (on_board yes) (fields_autoplaced)
     (property "Reference" "R11" (id 0) (at 72.39 68.58 90))
-    (property "Value" "330" (id 1) (at 72.39 71.12 90))
+    (property "Value" "220" (id 1) (at 72.39 71.12 90))
     (property "Footprint" "Resistor_THT:R_Axial_DIN0207_L6.3mm_D2.5mm_P15.24mm_Horizontal" (id 2) (at 72.39 73.152 90)
       (effects (font (size 1.27 1.27)) hide)
@@
     )
     (path "/902da62a-b458-446d-811e-6047e42b91c8"
-      (reference "R11") (unit 1) (value "330") (footprint "Resistor_THT:R_Axial_DIN0207_L6.3mm_D2.5mm_P15.24mm_Horizontal")
+      (reference "R11") (unit 1) (value "220") (footprint "Resistor_THT:R_Axial_DIN0207_L6.3mm_D2.5mm_P15.24mm_Horizontal")
     )
     (path "/4da6ace0-147e-454d-9d17-96e9dfa266de"
